Commit message: Preserve RSN FT model, planning configuration and SDK version

File: xarm_description/urdf/common/common.gazebo.xacro (robot description, xacro)
@@ -1,13 +1,4 @@
 <?xml version="1.0"?>
 <robot xmlns:xacro="http://ros.org/wiki/xacro">
-  <xacro:macro name="gz_ros2_control_plugin" params="ros2_control_params:=''">
-    <gazebo>
-      <plugin filename="gz_ros2_control-system" name="gz_ros2_control::GazeboSimROS2ControlPlugin">
-        <xacro:if value="${ros2_control_params != ''}">
-          <parameters>${ros2_control_params}</parameters>
-        </xacro:if>
-      </plugin>
-    </gazebo>
-  </xacro:macro>
   <xacro:macro name="ignition_ros2_control_plugin" params="prefix:='' ros2_control_params:=''">
     <gazebo>

File: xarm_description/urdf/common/common.link.xacro (robot description, xacro)
@@ -25,5 +25,4 @@
   </xacro:macro>
   <xacro:macro name="common_link_visual" params="mesh_filename add_mesh_suffix:=true material_name:='White' origin_xyz:='0 0 0' origin_rpy:='0 0 0' other_mesh_suffix:=''">
-    <xacro:property name="add_material" value="${mesh_suffix != 'dae'}"/>
     <visual>
       <geometry>
@@ -33,5 +32,4 @@
         <xacro:unless value="${add_mesh_suffix}">
           <xacro:if value="${other_mesh_suffix != ''}">
-            <xacro:property name="add_material" value="${other_mesh_suffix != 'dae'}"/>
             <mesh filename="${mesh_path}/${mesh_filename}.${other_mesh_suffix}"/>
           </xacro:if>
@@ -42,7 +40,5 @@
       </geometry>
       <origin xyz="${origin_xyz}" rpy="${origin_rpy}"/>
-      <xacro:if value="${add_material}">
-        <material name="${material_name}" />
-      </xacro:if>
+      <material name="${material_name}" />
     </visual>
   </xacro:macro>

File: xarm_description/urdf/gripper/xarm_gripper.gazebo.xacro (robot description, xacro)
@@ -2,5 +2,5 @@
 <robot xmlns:xacro="http://ros.org/wiki/xacro">
   <!-- from mimic_joint_gazebo_tutorial by @mintar, refer: https://github.com/mintar/mimic_joint_gazebo_tutorial -->
-  <xacro:macro name="mimic_joint_plugin_gazebo" params="name_prefix following_joint mimic_joint has_pid:=false multiplier:=1.0 offset:=0 sensitiveness:=0.0 max_effort:=1.0 ros2_control_plugin:='gazebo_ros2_control/GazeboSystem' robot_namespace:=''">
+  <xacro:macro name="mimic_joint_plugin_gazebo" params="name_prefix following_joint mimic_joint has_pid:=false multiplier:=1.0 offset:=0 sensitiveness:=0.0 max_effort:=1.0 robot_namespace:=''">
     <!-- ros2 -->
     <xacro:if value="${is_ros2}">
@@ -12,12 +12,6 @@
       <!-- <xacro:property name="filename" value="libroboticsgroup_upatras_gazebo_mimic_joint_plugin.so" /> -->
     </xacro:unless>
-    <xacro:if value="${ros2_control_plugin == 'gazebo_ros2_control/GazeboSystem'}">
-      <xacro:property name="plugin_name" value="${name_prefix}mimic_joint_plugin" />
-    </xacro:if>
-    <xacro:unless value="${ros2_control_plugin == 'gazebo_ros2_control/GazeboSystem'}">
-      <xacro:property name="plugin_name" value="gz::sim::systems::GazeboMimicJointPlugin" />
-    </xacro:unless>
     <gazebo>
-      <plugin name="${plugin_name}" filename="${filename}">
+      <plugin name="${name_prefix}mimic_joint_plugin" filename="${filename}">
         <joint>${following_joint}</joint>
         <mimicJoint>${mimic_joint}</mimicJoint>

File: xarm_description/urdf/gripper/xarm_gripper.urdf.xacro (robot description, xacro)
@@ -1,13 +1,5 @@
 <?xml version="1.0"?>
 <robot xmlns:xacro="http://ros.org/wiki/xacro" name="xarm_gripper">
-  <xacro:macro name="xarm_gripper_urdf" params="prefix:='' attach_to:='' attach_xyz:='0 0 0' attach_rpy:='0 0 0' gripper_version:='G1' ">
-    <xacro:property name="add_mesh_suffix" value="true"/>
-    <xacro:property name="other_mesh_suffix" value=""/>
-    <xacro:property name="name_suffix" value=""/>
-    <xacro:if value="${gripper_version == 'G2' or gripper_version == 'g2'}">
-      <xacro:property name="name_suffix" value="_g2"/>
-      <xacro:property name="other_mesh_suffix" value="dae"/>
-      <xacro:property name="add_mesh_suffix" value="false"/>
-    </xacro:if>
+  <xacro:macro name="xarm_gripper_urdf" params="prefix:='' attach_to:='' attach_xyz:='0 0 0' attach_rpy:='0 0 0' ">
     <xacro:unless value="${attach_to == ''}">
       <joint name="${prefix}gripper_fix" type="fixed">
@@ -26,14 +18,10 @@
       </inertial>
       <xacro:common_link_visual
-        mesh_filename="gripper/xarm/base_link${name_suffix}"
-        add_mesh_suffix="${add_mesh_suffix}"
-        other_mesh_suffix="${other_mesh_suffix}"
+        mesh_filename="gripper/xarm/base_link"
         origin_xyz="0 0 0"
         origin_rpy="0 0 0"
         material_name="${prefix}White" />
       <xacro:common_link_collision
-        mesh_filename="gripper/xarm/base_link${name_suffix}"
-        add_mesh_suffix="${add_mesh_suffix}"
-        other_mesh_suffix="${other_mesh_suffix}"
+        mesh_filename="gripper/xarm/base_link"
         origin_xyz="0 0 0"
         origin_rpy="0 0 0" />
@@ -48,14 +36,10 @@
       </inertial>
       <xacro:common_link_visual
-        mesh_filename="gripper/xarm/left_outer_knuckle${name_suffix}"
-        add_mesh_suffix="${add_mesh_suffix}"
-        other_mesh_suffix="${other_mesh_suffix}"
+        mesh_filename="gripper/xarm/left_outer_knuckle"
         origin_xyz="0 0 0"
         origin_rpy="0 0 0"
         material_name="${prefix}Silver" />
       <xacro:common_link_collision
-        mesh_filename="gripper/xarm/left_outer_knuckle${name_suffix}"
-        add_mesh_suffix="${add_mesh_suffix}"
-        other_mesh_suffix="${other_mesh_suffix}"
+        mesh_filename="gripper/xarm/left_outer_knuckle"
         origin_xyz="0 0 0"
         origin_rpy="0 0 0" />
@@ -77,14 +61,10 @@
       </inertial>
       <xacro:common_link_visual
-        mesh_filename="gripper/xarm/left_finger${name_suffix}"
-        add_mesh_suffix="${add_mesh_suffix}"
-        other_mesh_suffix="${other_mesh_suffix}"
+        mesh_filename="gripper/xarm/left_finger"
         origin_xyz="0 0 0"
         origin_rpy="0 0 0"
         material_name="${prefix}Silver" />
       <xacro:common_link_collision
-        mesh_filename="gripper/xarm/left_finger${name_suffix}"
-        add_mesh_suffix="${add_mesh_suffix}"
-        other_mesh_suffix="${other_mesh_suffix}"
+        mesh_filename="gripper/xarm/left_finger"
         origin_xyz="0 0 0"
         origin_rpy="0 0 0" />
@@ -107,14 +87,10 @@
       </inertial>
       <xacro:common_link_visual
-        mesh_filename="gripper/xarm/left_inner_knuckle${name_suffix}"
-        add_mesh_suffix="${add_mesh_suffix}"
-        other_mesh_suffix="${other_mesh_suffix}"
+        mesh_filename="gripper/xarm/left_inner_knuckle"
         origin_xyz="0 0 0"
         origin_rpy="0 0 0"
         material_name="${prefix}Silver" />
       <xacro:common_link_collision
-        mesh_filename="gripper/xarm/left_inner_knuckle${name_suffix}"
-        add_mesh_suffix="${add_mesh_suffix}"
-        other_mesh_suffix="${other_mesh_suffix}"
+        mesh_filename="gripper/xarm/left_inner_knuckle"
         origin_xyz="0 0 0"
         origin_rpy="0 0 0" />
@@ -137,14 +113,10 @@
       </inertial>
       <xacro:common_link_visual
-        mesh_filename="gripper/xarm/right_outer_knuckle${name_suffix}"
-        add_mesh_suffix="${add_mesh_suffix}"
-        other_mesh_suffix="${other_mesh_suffix}"
+        mesh_filename="gripper/xarm/right_outer_knuckle"
         origin_xyz="0 0 0"
         origin_rpy="0 0 0"
         material_name="${prefix}Silver" />
       <xacro:common_link_collision
-        mesh_filename="gripper/xarm/right_outer_knuckle${name_suffix}"
-        add_mesh_suffix="${add_mesh_suffix}"
-        other_mesh_suffix="${other_mesh_suffix}"
+        mesh_filename="gripper/xarm/right_outer_knuckle"
         origin_xyz="0 0 0"
         origin_rpy="0 0 0" />
@@ -167,14 +139,10 @@
       </inertial>
       <xacro:common_link_visual
-        mesh_filename="gripper/xarm/right_finger${name_suffix}"
-        add_mesh_suffix="${add_mesh_suffix}"
-        other_mesh_suffix="${other_mesh_suffix}"
+        mesh_filename="gripper/xarm/right_finger"
         origin_xyz="0 0 0"
         origin_rpy="0 0 0"
         material_name="${prefix}Silver" />
       <xacro:common_link_collision
-        mesh_filename="gripper/xarm/right_finger${name_suffix}"
-        add_mesh_suffix="${add_mesh_suffix}"
-        other_mesh_suffix="${other_mesh_suffix}"
+        mesh_filename="gripper/xarm/right_finger"
         origin_xyz="0 0 0"
         origin_rpy="0 0 0" />
@@ -197,14 +165,10 @@
       </inertial>
       <xacro:common_link_visual
-        mesh_filename="gripper/xarm/right_inner_knuckle${name_suffix}"
-        add_mesh_suffix="${add_mesh_suffix}"
-        other_mesh_suffix="${other_mesh_suffix}"
+        mesh_filename="gripper/xarm/right_inner_knuckle"
         origin_xyz="0 0 0"
         origin_rpy="0 0 0"
         material_name="${prefix}Silver" />
       <xacro:common_link_collision
-        mesh_filename="gripper/xarm/right_inner_knuckle${name_suffix}"
-        add_mesh_suffix="${add_mesh_suffix}"
-        other_mesh_suffix="${other_mesh_suffix}"
+        mesh_filename="gripper/xarm/right_inner_knuckle"
         origin_xyz="0 0 0"
         origin_rpy="0 0 0" />

File: xarm_description/urdf/gripper/xarm_gripper_macro.xacro (robot description, xacro)
@@ -7,9 +7,9 @@
   <xacro:include filename="$(find xarm_description)/urdf/gripper/xarm_gripper.gazebo.xacro" />
   <xacro:macro name="xarm_gripper_macro" params="prefix:='' attach_to:='' ns:='xarm' attach_xyz:='0 0 0' attach_rpy:='0 0 0'
-    ros2_control_plugin:='uf_robot_hardware/UFRobotFakeSystemHardware' dof:=7 hard_interface:='PositionJointInterface' gripper_version:='G1'"> ">
+    ros2_control_plugin:='uf_robot_hardware/UFRobotFakeSystemHardware' dof:=7 hard_interface:='PositionJointInterface' ">
     <xacro:if value="${is_ros2 and ros2_control_plugin != 'uf_robot_hardware/UFRobotSystemHardware'}">
       <xacro:xarm_gripper_ros2_control prefix="${prefix}" ros2_control_plugin="${ros2_control_plugin}" />
     </xacro:if>
-    <xacro:xarm_gripper_urdf prefix="${prefix}" attach_to="${attach_to}" attach_xyz="${attach_xyz}" attach_rpy="${attach_rpy}" gripper_version="${gripper_version}" />
+    <xacro:xarm_gripper_urdf prefix="${prefix}" attach_to="${attach_to}" attach_xyz="${attach_xyz}" attach_rpy="${attach_rpy}" />
     <xacro:xarm_gripper_transmission prefix="${prefix}" hard_interface="${hard_interface}" />
     <xacro:xarm_gripper_gazebo prefix="${prefix}" />
@@ -20,17 +20,17 @@
     <xacro:mimic_joint_plugin_gazebo name_prefix="${prefix}left_finger_joint"
       following_joint="${prefix}drive_joint" mimic_joint="${prefix}left_finger_joint"
-      has_pid="${is_ros2}" multiplier="1.0" max_effort="10.0" ros2_control_plugin="${ros2_control_plugin}"/>
+      has_pid="${is_ros2}" multiplier="1.0" max_effort="10.0" />
     <xacro:mimic_joint_plugin_gazebo name_prefix="${prefix}left_inner_knuckle_joint"
       following_joint="${prefix}drive_joint" mimic_joint="${prefix}left_inner_knuckle_joint"
-      has_pid="${is_ros2}" multiplier="1.0" max_effort="10.0" ros2_control_plugin="${ros2_control_plugin}"/>
+      has_pid="${is_ros2}" multiplier="1.0" max_effort="10.0" />
     <xacro:mimic_joint_plugin_gazebo name_prefix="${prefix}right_outer_knuckle_joint"
       following_joint="${prefix}drive_joint" mimic_joint="${prefix}right_outer_knuckle_joint"
-      has_pid="${is_ros2}" multiplier="1.0" max_effort="10.0" ros2_control_plugin="${ros2_control_plugin}"/>
+      has_pid="${is_ros2}" multiplier="1.0" max_effort="10.0" />
     <xacro:mimic_joint_plugin_gazebo name_prefix="${prefix}right_finger_joint"
       following_joint="${prefix}drive_joint" mimic_joint="${prefix}right_finger_joint"
-      has_pid="${is_ros2}" multiplier="1.0" max_effort="10.0" ros2_control_plugin="${ros2_control_plugin}"/>
+      has_pid="${is_ros2}" multiplier="1.0" max_effort="10.0" />
     <xacro:mimic_joint_plugin_gazebo name_prefix="${prefix}right_inner_knuckle_joint"
       following_joint="${prefix}drive_joint" mimic_joint="${prefix}right_inner_knuckle_joint"
-      has_pid="${is_ros2}" multiplier="1.0" max_effort="10.0" ros2_control_plugin="${ros2_control_plugin}"/>
+      has_pid="${is_ros2}" multiplier="1.0" max_effort="10.0" />
   </xacro:macro>
 </robot>

File: xarm_description/urdf/xarm7/xarm7.urdf.xacro (robot description, xacro)
@@ -13,5 +13,5 @@
     >
     <!-- define property -->
-    <xacro:if value="${mesh_suffix == 'dae' or (model_num >= 1305 and model_num != 1380)}">
+    <xacro:if value="${model_num >= 1305 and model_num != 1380}">
       <xacro:property name="visual_dir" value="xarm7_1305/visual"/>
       <xacro:property name="collision_dir" value="xarm7_1305/collision"/>
@@ -21,5 +21,5 @@
       <xacro:property name="link7_collision" value="xarm7_1305/collision/link7"/>
     </xacro:if>
-    <xacro:unless value="${mesh_suffix == 'dae' or (model_num >= 1305 and model_num != 1380)}">
+    <xacro:unless value="${model_num >= 1305 and model_num != 1380}">
       <xacro:property name="visual_dir" value="xarm7/visual"/>
       <xacro:property name="collision_dir" value="xarm7/visual"/>
@@ -275,4 +275,37 @@
       <dynamics damping="2" friction="1" />
     </joint>
+    <!-- FT sensor link -->
+    <link name="${prefix}ft_sensor_link">
+      <inertial>
+        <origin xyz="0 0 0" rpy="0 0 0" />
+        <mass value="0.2" />
+        <inertia
+          ixx="1e-4" ixy="0"   ixz="0"
+          iyy="1e-4" iyz="0"   izz="1e-4" />
+      </inertial>
+      <!-- 圆柱形的 FT 传感器 -->
+      <visual>
+        <!-- 这个 origin 先临时写 0，后面再调高度 -->
+        <origin xyz="0 0 0" rpy="0 0 0" />
+        <geometry>
+          <!-- radius / length 你可以根据实际 FT 传感器尺寸再微调 -->
+          <cylinder radius="0.035" length="0.025"/>
+        </geometry>
+        <material name="${prefix}Silver"/>
+      </visual>
+      <collision>
+        <origin xyz="0 0 0" rpy="0 0 0" />
+        <geometry>
+          <cylinder radius="0.03" length="0.03"/>
+        </geometry>
+      </collision>
+    </link>
+    <!-- FT sensor joint: 固定在 link7 上 -->
+    <joint name="${prefix}joint_ft_sensor" type="fixed">
+      <!-- z 轴方向往上（或者往下）挪一点，请你试着调这个数 -->
+      <origin xyz="0 0 0" rpy="0 0 0" />
+      <parent link="${prefix}link7" />
+      <child  link="${prefix}ft_sensor_link" />
+    </joint>
     <!-- <link name="${prefix}link_eef" />
     <joint name="${prefix}joint_eef" type="fixed">

File: xarm_description/urdf/xarm_device.urdf.xacro (robot description, xacro)
@@ -39,5 +39,4 @@
   <xacro:arg name="mesh_suffix" default="stl"/>
   <xacro:arg name="kinematics_suffix" default=""/>
-  <xacro:arg name="gripper_version" default="G1"/>
   <!-- load xarm device -->
   <xacro:include filename="$(find xarm_description)/urdf/xarm_device_macro.xacro" />
@@ -60,5 +59,4 @@
     baud_checkset="$(arg baud_checkset)" default_gripper_baud="$(arg default_gripper_baud)"
     model1300="$(arg model1300)" attach_to="$(arg attach_to)" attach_xyz="$(arg attach_xyz)" attach_rpy="$(arg attach_rpy)"
-    robot_sn="$(arg robot_sn)" use_gazebo_camera="$(arg use_gazebo_camera)" mesh_suffix="$(arg mesh_suffix)" kinematics_suffix="$(arg kinematics_suffix)"
-    gripper_version="$(arg gripper_version)" />
+    robot_sn="$(arg robot_sn)" use_gazebo_camera="$(arg use_gazebo_camera)" mesh_suffix="$(arg mesh_suffix)" kinematics_suffix="$(arg kinematics_suffix)" />
 </robot>

File: xarm_description/urdf/xarm_device_macro.xacro (robot description, xacro)
@@ -42,5 +42,4 @@
     mesh_suffix:='stl'
     kinematics_suffix:=''
-    gripper_version:='G1'
     "
     >
@@ -53,9 +52,9 @@
     <!-- Specify Mesh file path -->
     <xacro:property name="mesh_suffix" value="${mesh_suffix}" scope="parent"/>
-    <xacro:if value="${ros2_control_plugin == 'gazebo_ros2_control/GazeboSystem' or ros2_control_plugin == 'ign_ros2_control/IgnitionSystem' or ros2_control_plugin == 'gz_ros2_control/GazeboSimSystem'}">
+    <xacro:if value="${ros2_control_plugin == 'gazebo_ros2_control/GazeboSystem' or ros2_control_plugin == 'ign_ros2_control/IgnitionSystem'}">
       <!-- gazebo use -->
       <xacro:property name="mesh_path" value="file://$(find xarm_description)/meshes" scope="parent"/>
     </xacro:if>
-    <xacro:unless value="${ros2_control_plugin == 'gazebo_ros2_control/GazeboSystem' or ros2_control_plugin == 'ign_ros2_control/IgnitionSystem' or ros2_control_plugin == 'gz_ros2_control/GazeboSimSystem'}">
+    <xacro:unless value="${ros2_control_plugin == 'gazebo_ros2_control/GazeboSystem' or ros2_control_plugin == 'ign_ros2_control/IgnitionSystem'}">
       <xacro:property name="mesh_path" value="package://xarm_description/meshes" scope="parent"/>
     </xacro:unless>
@@ -208,18 +207,5 @@
       <xacro:if value="${add_d435i_links}">
         <xacro:include filename="$(find xarm_description)/urdf/camera/realsense.gazebo.xacro" />
-        <xacro:if value="${is_ros2}">
-          <xacro:if value="${ros2_control_plugin == 'gz_ros2_control/GazeboSimSystem'}">
-            <xacro:realsense_gz prefix="${prefix}" />
-          </xacro:if>
-          <xacro:if value="${ros2_control_plugin == 'ign_ros2_control/IgnitionSystem'}">
-            <xacro:realsense_ignition prefix="${prefix}" />
-          </xacro:if>
-          <xacro:if value="${ros2_control_plugin == 'gazebo_ros2_control/GazeboSystem'}">
-            <xacro:realsense_gazebo prefix="${prefix}" />
-          </xacro:if>
-        </xacro:if>
-        <xacro:unless value="${is_ros2}">
-          <xacro:realsense_gazebo prefix="${prefix}" />
-        </xacro:unless>
+        <xacro:realsense_gazebo prefix="${prefix}" />
       </xacro:if>
     </xacro:if>
@@ -235,15 +221,18 @@
       <xacro:if value="${robot_type == 'lite'}">
         <!-- Load Lite Gripper Model URDF -->
-        <xacro:include filename="$(find xarm_description)/urdf/gripper/uflite_gripper_macro.xacro" />
-        <xacro:uflite_gripper_macro prefix="${prefix}" attach_to="${prefix}link_eef"
-          ros2_control_plugin="${ros2_control_plugin}" dof="${dof}" hard_interface="${hard_interface}"
-          gripper_version="${gripper_version}" />
+        <xacro:include filename="$(find xarm_description)/urdf/gripper/lite_gripper.urdf.xacro" />
+        <xacro:uflite_gripper_urdf prefix="${prefix}" attach_to="${prefix}link_eef" />
       </xacro:if>
       <xacro:unless value="${robot_type == 'lite'}">
         <!-- Load XArm Gripper Model URDF -->
         <xacro:include filename="$(find xarm_description)/urdf/gripper/xarm_gripper_macro.xacro" />
+        <!-- attach_xyz="0 0 0.052" accounts for the FT sensor stacked between
+             link_eef (robot flange) and the xArm gripper. With this offset
+             link_tcp ends up 0.224 m from the flange, matching Studio's TCP
+             setting and removing the need for a runtime tcp_z_offset_m
+             compensation in xarm_controller_node. -->
         <xacro:xarm_gripper_macro prefix="${prefix}" attach_to="${prefix}link_eef"
-          ros2_control_plugin="${ros2_control_plugin}" dof="${dof}" hard_interface="${hard_interface}"
-          gripper_version="${gripper_version}" />
+          attach_xyz="0 0 0.052"
+          ros2_control_plugin="${ros2_control_plugin}" dof="${dof}" hard_interface="${hard_interface}" />
       </xacro:unless>
     </xacro:if>
@@ -253,6 +242,5 @@
         <xacro:include filename="$(find xarm_description)/urdf/gripper/bio_gripper_macro.xacro" />
         <xacro:bio_gripper_macro prefix="${prefix}" attach_to="${prefix}link_eef"
-          ros2_control_plugin="${ros2_control_plugin}" dof="${dof}" hard_interface="${hard_interface}"
-          gripper_version="${gripper_version}" />
+          ros2_control_plugin="${ros2_control_plugin}" dof="${dof}" hard_interface="${hard_interface}" />
       </xacro:unless>
     </xacro:if>

File: xarm_moveit_config/srdf/_xarm7_macro.srdf.xacro (robot description, xacro)
@@ -138,4 +138,13 @@
       <disable_collisions link1="${prefix}link_eef" link2="${prefix}right_outer_knuckle" reason="Never" />
       <disable_collisions link1="${prefix}link_eef" link2="${prefix}xarm_gripper_base_link" reason="Adjacent" />
+      <disable_collisions link1="${prefix}ft_sensor_link" link2="${prefix}xarm_gripper_base_link" reason="Adjacent" />
+      <disable_collisions link1="${prefix}ft_sensor_link" link2="${prefix}link7" reason="Adjacent" />
+      <disable_collisions link1="${prefix}ft_sensor_link" link2="${prefix}link_eef" reason="Adjacent" />
+      <disable_collisions link1="${prefix}ft_sensor_link" link2="${prefix}left_finger" reason="Never" />
+      <disable_collisions link1="${prefix}ft_sensor_link" link2="${prefix}left_inner_knuckle" reason="Never" />
+      <disable_collisions link1="${prefix}ft_sensor_link" link2="${prefix}left_outer_knuckle" reason="Never" />
+      <disable_collisions link1="${prefix}ft_sensor_link" link2="${prefix}right_finger" reason="Never" />
+      <disable_collisions link1="${prefix}ft_sensor_link" link2="${prefix}right_inner_knuckle" reason="Never" />
+      <disable_collisions link1="${prefix}ft_sensor_link" link2="${prefix}right_outer_knuckle" reason="Never" />
     </xacro:if>
     <!-- bio gripper -->
